File: turing_machine_driver/turing_driver.kicad_pcb (KiCad board)
At the start: 2 copper layers, 165.1 x 110.5 mm, 72 parts, among them J1 RPi Interface, J2 Header Position Value, J3 Symbol Register Value, J4 State Register Value, J5 External Interface, J6 Signal_connector_1, J7 Signal_connector_0, Q1 55NF06, U1 74LS14, U10 74LS245, U11 SST39SF020, U12 74LS245, U13 74LS245, U14 74LS245, U15 74LS245, U2 74LS03, U3 74LS04, U4 74LS139, U5 74LS74, U6 NE555P, U7 NE555P, U8 NE555P, U9 74LS245

Commit message: added github links to core and driver boards
Other:
- board text added: "https://github.com/szymanp135/Tura"
- board text removed: "Tura Paweł Szymański 02.2026"
Changed lines of the file:
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@@
 	(gr_rect
 		(start 106.045 131.445)
-		(end 119.126 135.89)
-		(stroke
-			(width 0.05)
-			(type solid)
-		)
-		(fill yes)
-		(layer "B.Cu")
-	)
-	(gr_rect
-		(start 119.126 135.509)
-		(end 182.88 135.89)
+		(end 183.261 135.89)
 		(stroke
 			(width 0.05)
@@
 		(layer "Edge.Cuts")
 	)
-	(gr_text "Tura    Paweł Szymański   02.2026"
-		(at 182.88 134.62 0)
-		(layer "B.Cu" knockout)
-		(effects
-			(font
-				(size 2.3 2.3)
-				(thickness 0.46)
-				(bold yes)
-			)
-			(justify left bottom mirror)
-		)
-	)
 	(gr_text "Paweł Szymański\n02.2026"
 		(at 184.15 100.33 0)
@@
 		)
 	)
+	(gr_text "https://github.com/szymanp135/Tura"
+		(at 181.61 134.62 0)
+		(layer "B.SilkS")
+		(effects
+			(font
+				(size 2 2)
+				(thickness 0.25)
+			)
+			(justify left bottom mirror)
+		)
+	)

Commit message: added backplane PCB and adjusted driver silkscreen text thickness
Changed lines of the file:
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@@
 			(font
 				(size 1.5 1.5)
-				(thickness 0.3)
+				(thickness 0.25)
 				(bold yes)
 			)
@@
 			(font
 				(size 1.6 1.6)
-				(thickness 0.32)
+				(thickness 0.3)
 				(bold yes)
 			)
@@
 			(font
 				(size 5 5)
-				(thickness 0.625)
+				(thickness 0.7)
 			)
 			(justify left bottom)
